Commit message: slam, speech

File: install/rafeeq_description/share/rafeeq_description/urdf/robot_description.urdf (robot description, URDF)
Before this commit: robot rafeeq, 10 links, 9 joints
Links:
- added link base_footprint
Joints:
- added joint base_footprint_joint: type fixed, parent base_footprint, child base_link, origin xyz=0 0 0.456 rpy=0 0 0

Commit message: slam_and_navigation_edits

File: install/rafeeq_description/share/rafeeq_description/urdf/robot_description.urdf (robot description, URDF)
Before this commit: robot rafeeq, 11 links, 10 joints
Links:
- link base_link: mass 68.5887337151705 -> 15
Joints:
- joint LeftMotor_joint: origin xyz=-0.30241 0.17408 -0.35719 rpy=1.5708 0 0 -> xyz=-0.30241 0.17408 -0.2 rpy=1.5708 0 0
- joint RightMotor_joint: origin xyz=-0.30241 -0.17408 -0.35719 rpy=1.5708 0 0 -> xyz=-0.30241 -0.17408 -0.2 rpy=1.5708 0 0
